Commit message: added collision and g = -9.81 (Anna would be proud)

File: Simulation/models/crab_model.urdf (robot description, URDF)
Before this commit: robot crab, 32 links, 31 joints
Links:
- link coxa_l1: geometry collision mesh filename=meshes/coxa_l.STL; visual mesh filename=meshes/coxa_l.STL
- link coxa_l2: geometry collision mesh filename=meshes/coxa_l.STL; visual mesh filename=meshes/coxa_l.STL
- link coxa_l3: geometry collision mesh filename=meshes/coxa_l.STL; visual mesh filename=meshes/coxa_l.STL
- link coxa_r1: geometry collision mesh filename=meshes/coxa_r.STL; visual mesh filename=meshes/coxa_r.STL
- link coxa_r2: geometry collision mesh filename=meshes/coxa_r.STL; visual mesh filename=meshes/coxa_r.STL
- link coxa_r3: geometry collision mesh filename=meshes/coxa_r.STL; visual mesh filename=meshes/coxa_r.STL
- link femur_l1: geometry collision mesh filename=meshes/femur_l.STL; visual mesh filename=meshes/femur_l.STL
- link femur_l2: geometry collision mesh filename=meshes/femur_l.STL; visual mesh filename=meshes/femur_l.STL
- link femur_l3: geometry collision mesh filename=meshes/femur_l.STL; visual mesh filename=meshes/femur_l.STL
- link femur_r1: geometry collision mesh filename=meshes/femur_r.STL; visual mesh filename=meshes/femur_r.STL
- link femur_r2: geometry collision mesh filename=meshes/femur_r.STL; visual mesh filename=meshes/femur_r.STL
- link femur_r3: geometry collision mesh filename=meshes/femur_r.STL; visual mesh filename=meshes/femur_r.STL
- link thorax: geometry collision mesh filename=meshes/thorax.STL; visual mesh filename=meshes/thorax.STL
- link tibia_l1: geometry collision mesh filename=meshes/tibia_l.STL; visual mesh filename=meshes/tibia_l.STL
- link tibia_l2: geometry collision mesh filename=meshes/tibia_l.STL; visual mesh filename=meshes/tibia_l.STL
- link tibia_l3: geometry collision mesh filename=meshes/tibia_l.STL; visual mesh filename=meshes/tibia_l.STL
- link tibia_r1: geometry collision mesh filename=meshes/tibia_r.STL; visual mesh filename=meshes/tibia_r.STL
- link tibia_r2: geometry collision mesh filename=meshes/tibia_r.STL; visual mesh filename=meshes/tibia_r.STL
- link tibia_r3: geometry collision mesh filename=meshes/tibia_r.STL; visual mesh filename=meshes/tibia_r.STL
